File: WSController.sch (KiCad schematic (older format))
At the start: 19 parts, among them J1 AVR-ISP-6, J2 LED Strip, Q1 IRLR024N, Q2 BC857, Q3 IRLR024N, SW1 Switch Mode, SW2 Switch ON, U1 ATmega328P-AU

Commit message: corrected values of R4 and R5
Parts:
- R4: value 10k -> 1k
- R5: value 1k -> 10k
Changed lines of the file:
@@
 EESchema Schematic File Version 4
-LIBS:WSController-cache
 EELAYER 30 0
 EELAYER END
@@
 P 7450 3300
 F 0 "R4" H 7520 3346 50  0000 L CNN
-F 1 "10k" H 7520 3255 50  0000 L CNN
+F 1 "1k" H 7520 3255 50  0000 L CNN
 F 2 "Resistor_SMD:R_0805_2012Metric_Pad1.15x1.40mm_HandSolder" V 7380 3300 50  0001 C CNN
 F 3 "~" H 7450 3300 50  0001 C CNN
@@
 P 7450 3800
 F 0 "R5" H 7520 3846 50  0000 L CNN
-F 1 "1k" H 7520 3755 50  0000 L CNN
+F 1 "10k" H 7520 3755 50  0000 L CNN
 F 2 "Resistor_SMD:R_0805_2012Metric_Pad1.15x1.40mm_HandSolder" V 7380 3800 50  0001 C CNN
 F 3 "~" H 7450 3800 50  0001 C CNN
